File: KiCAD/4mm_6mm_COUPLING_LOOP/4mm_6mm_COUPLING_LOOP.kicad_pcb (KiCad board)
At the start: 2 copper layers, 7.2 x 10.2 mm, 1 part

Commit message: Remove Bridge12 branding from KiCAD files and README
The EPR business of Bridge12 was acquired by Bruker in October 2024.
Remove all Bridge12/B12T references from the KiCad projects:
- Delete the Bridge12 logo footprint (b12t-logo-lowres) etched into the
  TOP and BOTTOM boards' silkscreen
- Rename the footprint library B12T_Open_PCB_LGR -> OpenPCBLGR (the
  library nickname, folder, and all footprint references across the
  four projects)
- Clear the "Bridge12 Technologies, Inc." company field from all
  schematic and PCB title blocks
- Drop the now-unused Bridge12 link from README.md

Co-Authored-By: Claude Sonnet 5 <noreply@anthropic.com>
Parts:
- AE1: footprint B12T_Open_PCB_LGR:4mm_Offset_6mm_Diameter_141-Semi-Rigid_Coupling_Loop -> OpenPCBLGR:4mm_Offset_6mm_Diameter_141-Semi-Rigid_Coupling_Loop
Changed lines of the file:
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@@
     (date 2022-07-15)
     (rev 1.0)
-    (company "Bridge12 Technologies, Inc.")
+    (company "")
     (comment 1 "X-Band Loop Gap Resonator Coupling Loop")
     (comment 4 "Timothy Keller")
@@
     (add_net "Net-(AE1-Pad1)")
   )
-  (module B12T_Open_PCB_LGR:4mm_Offset_6mm_Diameter_141-Semi-Rigid_Coupling_Loop (layer F.Cu)
+  (module OpenPCBLGR:4mm_Offset_6mm_Diameter_141-Semi-Rigid_Coupling_Loop (layer F.Cu)
     (at 100 100)
     (fp_text reference AE1 (at 5.08 3.81) (layer F.SilkS) hide
