File: KiCAD/5mm_X-Band_LGR/X-Band_EPR_LGR.kicad_pcb (KiCad board)
At the start: 2 copper layers, 31.8 x 31.8 mm, 5 parts

Commit message: Remove Bridge12 branding from KiCAD files and README
The EPR business of Bridge12 was acquired by Bruker in October 2024.
Remove all Bridge12/B12T references from the KiCad projects:
- Delete the Bridge12 logo footprint (b12t-logo-lowres) etched into the
  TOP and BOTTOM boards' silkscreen
- Rename the footprint library B12T_Open_PCB_LGR -> OpenPCBLGR (the
  library nickname, folder, and all footprint references across the
  four projects)
- Clear the "Bridge12 Technologies, Inc." company field from all
  schematic and PCB title blocks
- Drop the now-unused Bridge12 link from README.md

Co-Authored-By: Claude Sonnet 5 <noreply@anthropic.com>
Parts:
- H1: footprint B12T_Open_PCB_LGR:5.2mm_3L2G_X-Band -> OpenPCBLGR:5.2mm_3L2G_X-Band
Changed lines of the file:
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@@
     (date 2022-07-15)
     (rev 1.0)
-    (company "Bridge12 Technologies, Inc.")
+    (company "")
     (comment 1 "X-Band Loop Gap Resonator")
     (comment 4 "Timothy Keller")
@@
       (net 1 GND))
   )
-  (module B12T_Open_PCB_LGR:5.2mm_3L2G_X-Band (layer F.Cu)
+  (module OpenPCBLGR:5.2mm_3L2G_X-Band (layer F.Cu)
     (at 100 100)
     (fp_text reference H1 (at 1.27 -6.35) (layer F.SilkS) hide
