File: KiCAD/5mm_X-Band_LGR_BOTTOM/X-Band_EPR_LGR_BOTTOM.kicad_pcb (KiCad board)
At the start: 2 copper layers, 31.8 x 31.8 mm, 6 parts

Commit message: Remove Bridge12 branding from KiCAD files and README
The EPR business of Bridge12 was acquired by Bruker in October 2024.
Remove all Bridge12/B12T references from the KiCad projects:
- Delete the Bridge12 logo footprint (b12t-logo-lowres) etched into the
  TOP and BOTTOM boards' silkscreen
- Rename the footprint library B12T_Open_PCB_LGR -> OpenPCBLGR (the
  library nickname, folder, and all footprint references across the
  four projects)
- Clear the "Bridge12 Technologies, Inc." company field from all
  schematic and PCB title blocks
- Drop the now-unused Bridge12 link from README.md

Co-Authored-By: Claude Sonnet 5 <noreply@anthropic.com>
Parts:
- removed LOGO: Val**, B12T_Open_PCB_LGR:b12t-logo-lowres
